Commit message: fix MDH

File: my_robot/robot.urdf (robot description, URDF)
Before this commit: robot my_robot, 5 links, 4 joints
Joints:
- joint joint_1_joint: origin xyz=0 0 0 rpy=0 0 0 -> xyz=0 0 0.51 rpy=0 0 0
- joint joint_2_joint: origin xyz=0 0 0.51 rpy=1.5708 0 0 -> xyz=0 0 0 rpy=1.5708 0 0

Commit message: The MDH and viewer is the same as sketch now.

File: my_robot/robot.urdf (robot description, URDF)
Before this commit: robot my_robot, 5 links, 4 joints
Joints:
- joint joint_2_joint: origin xyz=0 0 0 rpy=1.5708 0 0 -> xyz=0 0 0 rpy=0 -1.5707963267948966 1.5707963267948966
- joint joint_3_joint: origin xyz=0.099988 0.0015514 0 rpy=1.5708 0 1.5708 -> xyz=0 -0.099988 -0.0015514 rpy=1.5707963267948966 0 0
